Commit message: ani

File: simulation_ws/src/ros2_robot_simulation/models/urdf/jetbot.urdf (robot description, URDF)
Before this commit: robot JetBot, 5 links, 4 joints
Joints:
- joint camera_joint: axis 0.96891  0       0.2474 -> 0.96891 0 0.2474; origin xyz=0.065   0      0.0857 rpy=0    0.25  0 -> xyz=0.065 0 0.0857 rpy=0 0.25 0
- joint left_wheel_hinge: axis 1  0  0 -> 1 0 0; origin xyz=0.03     0.05125  0.03 rpy=0       0       1.57079 -> xyz=0.03 0.05125 0.03 rpy=0 0 1.57079
- joint right_wheel_hinge: axis 1  0  0 -> 1 0 0; origin xyz=0.03   -0.0595  0.03 rpy=0       0       1.57079 -> xyz=0.03 -0.0595 0.03 rpy=0 0 1.57079
